Commit message: Modified boat_multi.launch to allow for positional and angular control of the boat model using a controller

File: fcu_sim/agents/boat/boat.xacro (robot description, xacro)
@@ -1,7 +1,3 @@
 <?xml version="1.0"?>
-<!--
-Gazebo Multirotor Definition File
-Author: James Jackson
--->
 <robot name="boat" xmlns:xacro="http://ros.org/wiki/xacro">
   <!-- Properties -->
@@ -9,9 +5,9 @@
   <xacro:property name="use_mesh_file" value="true" />
   <xacro:property name="mesh_file" value="package://fcu_sim/meshes/Boat/boat.dae" />
-  <xacro:property name="mass" value="2.856" />
+  <xacro:property name="mass" value="2.0" />
   <xacro:property name="body_width" value="0.505" />
   <xacro:property name="body_height" value="0.1" />
   <xacro:property name="body_inertia">
-    <inertia ixx="0.07" ixy="0.0" ixz="0.0" iyy="0.08" iyz="0.0" izz="0.12" />
+    <inertia ixx="0.05" ixy="0.0" ixz="0.0" iyy="0.05" iyz="0.0" izz="0.05" />
   </xacro:property>
   <!-- *********************** GAZEBO ROBOT DEFINITION ******************* -->
@@ -19,5 +15,5 @@
     <inertial>
       <mass value="${mass}" />  <!-- [kg] -->
-      <origin xyz="0 0 0" />
+      <origin xyz="10 0 0" />
       <xacro:insert_block name="body_inertia" />
     </inertial>
@@ -45,14 +41,29 @@
   <!-- ************************* FORCES AND MOMENTS ********************** -->
   <!-- ROSflight_SIL -->
-  <xacro:include filename="$(find fcu_sim_plugins)/xacro/ROSflight_SIL.xacro"/>
-  <!-- <xacro:mikey_ROSflight_SIL namespace="${namespace}" parent_link="${namespace}/base_link" command_topic="command"/> -->
-  <!-- Simplified Dynamics -->
-  <!-- <xacro:include filename="$(find fcu_sim_plugins)/xacro/multirotor_forces_and_moments.xacro"/>
-  <xacro:multirotor namespace="${namespace}" parent_link="${namespace}/base_link" command_topic="command"/>   -->
+  <!--<xacro:include filename="$(find fcu_sim_plugins)/xacro/ROSflight_SIL.xacro"/>-->
+  <xacro:include filename="$(find fcu_sim_plugins)/xacro/boat_forces_and_moments.xacro"/>
+  <xacro:boat_controller
+  	namespace="${namespace}"
+  	command_topic="boat_command"/>
+  <!-- ************************ GIMBAL COMMANDER ********************** -->
+  <!-- should not be used; does not move the boat but rather a hypothetical camera
+       according to the boat's orientation.
+  <xacro:include filename="$(find fcu_sim_plugins)/xacro/boat_tow.xacro"/>
+  <xacro:gimbal_BOAT
+  	namespace="${namespace}"
+  	parent_link="${namespace}/base_link"
+  	camera_topic="${namespace}/boatcam/data"
+  	frame_rate="1"
+  	pose_topic="${namespace}/boatpose"
+  	command_topic="${namespace}/boat_command"
+  	use_slipring="true">
+  	<origin xyz="10 0 0" rpy="0 0 0"/>
+  </xacro:gimbal_BOAT> -->
   <!-- ***************** SENSORS ******************* -->
-  <!-- Ground Truth -->
+  <!-- Ground Truth (Odometry plugin gets orientation info from gazebo and publishes it
+  		on the ROS network (as /.../ground_truth/odometry)-->
   <xacro:include filename="$(find fcu_sim_plugins)/xacro/odometry_sensor.xacro"/>
   <xacro:ground_truth namespace="${namespace}" parent_link="${namespace}/base_link" />
-  <!-- Mount an IMU -->
+  <!-- Mount an IMU (not being used when you have odometry plugin)-->
   <xacro:include filename="$(find fcu_sim_plugins)/xacro/imu.xacro"/>
   <xacro:perfect_IMU
@@ -60,32 +71,3 @@
     parent_link="${namespace}/base_link"
     imu_topic="imu/data"/>
-  <!--Enable Wind -->
- <!--  <xacro:include filename="$(find fcu_sim_plugins)/xacro/wind.xacro"/>
-  <xacro:wind_param
-    namespace="${namespace}"
-    link_name="${namespace}/base_link"
-    wind_pub_topic="wind"/> -->
-  <!-- Mount an Altimeter -->
-  <!-- <xacro:include filename="$(find fcu_sim_plugins)/xacro/sonar.xacro"/>
-  <xacro:Sonar_MB1030
-    namespace="${namespace}"
-    parent_link="${namespace}/base_link"
-    sonar_topic="alt">
-    <origin xyz="0 0 0" rpy="0 1.57 0" />
-  </xacro:Sonar_MB1030> -->
-  <!-- Mount an RGBD Camera -->
- <!--  <xacro:include filename="$(find fcu_sim_plugins)/xacro/rgbd.xacro"/>
-  <xacro:xtion
-    namespace="${namespace}"
-    parent_link="${namespace}/base_link"/> -->
-  <!-- Laser Scanner -->
-  <!-- <xacro:include filename="$(find fcu_sim_plugins)/xacro/laser_scanner.xacro"/>
-  <xacro:RPLIDAR-A2
-    namespace="${namespace}"
-    parent_link="${namespace}/base_link"
-    visualize="false">
-    <origin xyz="0.0 0.0 0.2" rpy="0 0 0" />
-  </xacro:RPLIDAR-A2> -->
-    <!-- Collision Sensor -->
-    <!-- TODO  http://gazebosim.org/tutorials?tut=contact_sensor-->
 </robot>

Commit message: Altered paths for smooth camera recording

File: fcu_sim/agents/boat/boat.xacro (robot description, xacro)
@@ -19,5 +19,5 @@
     </inertial>
     <visual>
-      <origin xyz="0 0 0" rpy="0 0 0" />
+      <origin xyz="10 0 0" rpy="0 0 0" />
       <geometry>
         <xacro:if value="${use_mesh_file}">
@@ -30,5 +30,5 @@
     </visual>
     <collision>
-      <origin xyz="0 0 0" rpy="0 0 0" />
+      <origin xyz="10 0 0" rpy="0 0 0" />
       <geometry>
         <cylinder length="${body_height}" radius="${body_width}"/>

Commit message: Added ArUco tags, made togglable options in a yaml file

File: fcu_sim/agents/boat/boat.xacro (robot description, xacro)
@@ -2,33 +2,37 @@
 <robot name="boat" xmlns:xacro="http://ros.org/wiki/xacro">
   <!-- Properties -->
-  <xacro:property name="namespace" value="boat" />
+	<xacro:property name="boat_dict" value="${load_yaml('boat.yaml')}" />
+	<xacro:property name="boat_type" value="${boat_dict['boat_type']}" />
+	<xacro:property name="aruco_num" value="${boat_dict['aruco_num']}" />
+	<xacro:property name="namespace" value="boat" />
   <xacro:property name="use_mesh_file" value="true" />
-  <xacro:property name="mesh_file" value="package://fcu_sim/meshes/Boat/boat.dae" />
-  <xacro:property name="mass" value="2.0" />
-  <xacro:property name="body_width" value="0.505" />
-  <xacro:property name="body_height" value="0.1" />
+  <xacro:property name="mesh_file" value="package://fcu_sim/meshes/Boat/${boat_type}_boat.dae" />
+	<xacro:property name="aruco_mesh_file_1" value="package://fcu_sim/meshes/Boat/arucos/aruco${aruco_num}.dae" /> <!--aruco4 doesn't work for some reason...-->
+  <xacro:property name="body_width" value="0.505" /> <!--+++++++++++++++++++-->
+  <xacro:property name="body_height" value="0.1" />  <!--+++++++++++++++++++-->
   <xacro:property name="body_inertia">
     <inertia ixx="0.05" ixy="0.0" ixz="0.0" iyy="0.05" iyz="0.0" izz="0.05" />
   </xacro:property>
   <!-- *********************** GAZEBO ROBOT DEFINITION ******************* -->
+  <!-- Define the base link, which represents the boat itself -->
   <link name="${namespace}/base_link">
     <inertial>
-      <mass value="${mass}" />  <!-- [kg] -->
-      <origin xyz="10 0 0" />
+      <mass value="${boat_dict['boat_mass']}" />  <!-- [kg] -->
+      <origin xyz="0 0 0" />
       <xacro:insert_block name="body_inertia" />
     </inertial>
-    <visual>
-      <origin xyz="10 0 0" rpy="0 0 0" />
-      <geometry>
-        <xacro:if value="${use_mesh_file}">
-          <mesh filename="${mesh_file}" scale="0.25 0.25 0.25" />
-        </xacro:if>
-        <xacro:unless value="${use_mesh_file}">
-          <cylinder length="${body_height}" radius="${body_width}"/>
-        </xacro:unless>
+		<visual>
+			<origin xyz="0 0 0" rpy="0 0 0" />
+			<geometry>
+        <xacro:if value="${boat_type == 'patrol'}">
+          <mesh filename="${mesh_file}" scale="0.55 0.55 0.55" />
+				</xacro:if>
+        <xacro:if value="${boat_type == 'pontoon'}">
+					<mesh filename="${mesh_file}" scale="1 1 1" />
+				</xacro:if>
       </geometry>
-    </visual>
+		</visual>
     <collision>
-      <origin xyz="10 0 0" rpy="0 0 0" />
+      <origin xyz="0 0 0" rpy="0 0 0" />
       <geometry>
         <cylinder length="${body_height}" radius="${body_width}"/>
@@ -36,28 +40,30 @@
     </collision>
   </link>
+  <!-- Define the aruco link, which is attached to the base link via a rigid joint -->
+  <link name="${namespace}/aruco_link_1">
+    <visual>
+			<xacro:if value="${boat_type == 'patrol'}">
+				<origin xyz="0 -3.5 -0.2" rpy="0 0 0" />
+			</xacro:if>
+			<xacro:if value="${boat_type == 'pontoon'}">
+				<origin xyz="0 -1.5 0.225" rpy="0 0 0" />
+			</xacro:if>
+			<geometry>
+				<mesh filename="${aruco_mesh_file_1}" scale="1.4 1.4 1.4" />
+			</geometry>
+		</visual>
+	</link>
+	<joint name="boat_to_aruco_1" type="fixed">
+		<parent link="${namespace}/base_link"/>
+		<child link="${namespace}/aruco_link_1"/>
+	</joint>
   <gazebo reference="${namespace}/base_link">
     <material>Gazebo/$(arg color)</material>
   </gazebo>
   <!-- ************************* FORCES AND MOMENTS ********************** -->
-  <!-- ROSflight_SIL -->
-  <!--<xacro:include filename="$(find fcu_sim_plugins)/xacro/ROSflight_SIL.xacro"/>-->
   <xacro:include filename="$(find fcu_sim_plugins)/xacro/boat_forces_and_moments.xacro"/>
   <xacro:boat_controller
   	namespace="${namespace}"
   	command_topic="boat_command"/>
-  <!-- ************************ GIMBAL COMMANDER ********************** -->
-  <!-- should not be used; does not move the boat but rather a hypothetical camera
-       according to the boat's orientation.
-  <xacro:include filename="$(find fcu_sim_plugins)/xacro/boat_tow.xacro"/>
-  <xacro:gimbal_BOAT
-  	namespace="${namespace}"
-  	parent_link="${namespace}/base_link"
-  	camera_topic="${namespace}/boatcam/data"
-  	frame_rate="1"
-  	pose_topic="${namespace}/boatpose"
-  	command_topic="${namespace}/boat_command"
-  	use_slipring="true">
-  	<origin xyz="10 0 0" rpy="0 0 0"/>
-  </xacro:gimbal_BOAT> -->
   <!-- ***************** SENSORS ******************* -->
   <!-- Ground Truth (Odometry plugin gets orientation info from gazebo and publishes it

Commit message: semi-functional waypoint following

File: fcu_sim/agents/boat/boat.xacro (robot description, xacro)
@@ -44,8 +44,8 @@
     <visual>
 			<xacro:if value="${boat_type == 'patrol'}">
-				<origin xyz="0 -3.5 -0.2" rpy="0 0 0" />
+				<origin xyz="3.5 0 -0.2" rpy="0 0 0" />
 			</xacro:if>
 			<xacro:if value="${boat_type == 'pontoon'}">
-				<origin xyz="0 -1.5 0.225" rpy="0 0 0" />
+				<origin xyz="1.75 0 0.225" rpy="0 0 0" />
 			</xacro:if>
 			<geometry>
